File: eurorack-smd-15v/juno-chorus-clone.kicad_pcb (KiCad board)
At the start: 2 copper layers, 59.1 x 108.5 mm, 168 parts, among them J1 +-15v In, P2 AUDIO_IN, P3 OUT_L, P4 Out_R, Q1 2SC1815, Q10 2SC1815, Q11 2SA1015, Q12 2SA1015, Q13 2SC1815, Q14 2SA1015, Q15 2SA1015, Q16 2SK30, Q18 2SA1015, Q19 2SA1015, Q2 2SC1815, Q20 2SK30, Q3 2SA1015, Q4 2SA1015, Q5 2SC1815, Q6 2SC1815, Q7 2SA1015, Q8 2SA1015, Q9 2SC1815, SW1 SW_PUSH, U1 TL084HID, U11 TL084HID, U5 MN3009, U6 MN3101, U7 MN3009, U8 MN3101

Commit message: Add Eurorack-style Panel
Parts:
- RV1: value 100k -> Rate 100k
- RV2: value 100k -> Depth 100k
- RV5: value 100k -> Input 100k
Changed lines of the file:
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@@
 			)
 		)
-		(property "Value" "100k"
+		(property "Value" "Depth 100k"
 			(at 2.5 4.6 90)
 			(layer "F.Fab")
@@
 			)
 		)
-		(property "Value" "100k"
+		(property "Value" "Rate 100k"
 			(at 2.5 4.6 90)
 			(layer "F.Fab")
@@
 			)
 		)
-		(property "Value" "100k"
+		(property "Value" "Input 100k"
 			(at 2.5 4.6 0)
 			(layer "F.Fab")

Commit message: Replace TL084 with TL074 to stay consistent with my other designs
Parts:
- U1, U11: value TL084HID -> TL074HID
Changed lines of the file:
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@@
 			)
 		)
-		(property "Value" "TL084HID"
+		(property "Value" "TL074HID"
 			(at 0 5.28 0)
 			(layer "F.Fab")
@@
 			)
 		)
-		(property "Value" "TL084HID"
+		(property "Value" "TL074HID"
 			(at 0 -5.28 90)
 			(layer "B.Fab")
